Commit message: Multi spawn ability

File: my_p2os/defs/pioneer3at.xacro (robot description, xacro)
@@ -5,5 +5,5 @@
        xmlns:xacro="http://ros.org/wiki/xacro"
        name="pioneer3at">
-<!-- <xacro:include filename="$(find my_p2os)/defs/pioneer3at_body.xacro"/> -->
+<xacro:arg name="namespace" default=""/>
 <xacro:include filename="$(find my_p2os)/defs/pioneer3at_body.xacro"/>
 <xacro:include filename="$(find my_p2os)/defs/hokuyo_utm30lx.urdf.xacro"/>

File: my_p2os/defs/pioneer3at_body.xacro (robot description, xacro)
@@ -17,5 +17,5 @@
 			<origin xyz="0 0 0.177" rpy="0 0 0"/>
 			<geometry name="pioneer_geom">
-				<mesh filename="package://p2os_urdf/meshes/p3at_meshes/chassis.stl"/>
+				<mesh filename="package://my_p2os/meshes/p3at_meshes/chassis.stl"/>
 			</geometry>
 			<material name="ChassisRed">
@@ -26,5 +26,5 @@
 			<origin xyz="0 0 0.177" rpy="0 0 0"/>
 				<geometry>
-					<mesh filename="package://p2os_urdf/meshes/p3at_meshes/chassis.stl"/>
+					<mesh filename="package://my_p2os/meshes/p3at_meshes/chassis.stl"/>
 				</geometry>
 		</collision>
@@ -45,5 +45,5 @@
 			<origin xyz="0 0 0" rpy="0 0 0"/>
 			<geometry name="pioneer_geom">
-				<mesh filename="package://p2os_urdf/meshes/p3at_meshes/top.stl"/>
+				<mesh filename="package://my_p2os/meshes/p3at_meshes/top.stl"/>
 			</geometry>
 			<material name="TopBlack">
@@ -77,5 +77,5 @@
 			<origin xyz="0 0 0" rpy="0 0 0"/>
 			<geometry name="pioneer_geom">
-				<mesh filename="package://p2os_urdf/meshes/p3at_meshes/front_sonar.stl"/>
+				<mesh filename="package://my_p2os/meshes/p3at_meshes/front_sonar.stl"/>
 			</geometry>
 			<material name="SonarYellow">
@@ -108,5 +108,5 @@
 			<origin xyz="0 0 0" rpy="0 0 0"/>
 			<geometry name="pioneer_geom">
-				<mesh filename="package://p2os_urdf/meshes/p3at_meshes/back_sonar.stl"/>
+				<mesh filename="package://my_p2os/meshes/p3at_meshes/back_sonar.stl"/>
 			</geometry>
 			<material name="SonarYellow">
@@ -141,5 +141,5 @@
 		<origin xyz="0 0 0" rpy="0 0 0"/>
 		<geometry name="pioneer_geom">
-			<mesh filename="package://p2os_urdf/meshes/p3at_meshes/axle.stl"/>
+			<mesh filename="package://my_p2os/meshes/p3at_meshes/axle.stl"/>
 		</geometry>
 		<material name="AxleGrey">
@@ -172,5 +172,5 @@
 		<origin xyz="0 0 0" rpy="0 0 0"/>
 		<geometry name="pioneer_geom">
-			<mesh filename="package://p2os_urdf/meshes/p3at_meshes/${suffix}_hubcap.stl"/>
+			<mesh filename="package://my_p2os/meshes/p3at_meshes/${suffix}_hubcap.stl"/>
 		</geometry>
 		<material name="HubcapYellow">
@@ -203,5 +203,5 @@
 		<origin xyz="0 0 0" rpy="0 0 0"/>
 		<geometry name="pioneer_geom">
-			<mesh filename="package://p2os_urdf/meshes/p3at_meshes/wheel.stl"/>
+			<mesh filename="package://my_p2os/meshes/p3at_meshes/wheel.stl"/>
 		</geometry>
 		<material name="WheelBlack">
@@ -212,5 +212,5 @@
 		<origin xyz="0 0 0" rpy="${-3.1415927/2} 0 0"/>
 		<geometry>
-	    <!--mesh filename="package://p2os_urdf/meshes/p3at_meshes/wheel.stl"/-->
+	    <!--mesh filename="package://my_p2os/meshes/p3at_meshes/wheel.stl"/-->
 	    <cylinder radius="0.111" length="0.075"/>
 		</geometry>
@@ -242,5 +242,5 @@
 		<origin xyz="0 0 0" rpy="0 0 0"/>
 		<geometry name="pioneer_geom">
-			<mesh filename="package://p2os_urdf/meshes/p3at_meshes/axle.stl"/>
+			<mesh filename="package://my_p2os/meshes/p3at_meshes/axle.stl"/>
 		</geometry>
 		<material name="AxleGrey">
@@ -251,5 +251,5 @@
 		<origin xyz="0 0 0" rpy="0 0 0"/>
 		<geometry>
-			<mesh filename="package://p2os_urdf/meshes/p3at_meshes/axle.stl"/>
+			<mesh filename="package://my_p2os/meshes/p3at_meshes/axle.stl"/>
 		</geometry>
 	</collision>
@@ -273,5 +273,5 @@
 		<origin xyz="0 0 0" rpy="0 0 0"/>
 		<geometry name="pioneer_geom">
-			<mesh filename="package://p2os_urdf/meshes/p3at_meshes/${suffix}_hubcap.stl"/>
+			<mesh filename="package://my_p2os/meshes/p3at_meshes/${suffix}_hubcap.stl"/>
 		</geometry>
 		<material name="HubcapYellow"/>
@@ -280,5 +280,5 @@
 		<origin xyz="0 0 0" rpy="0 0 0"/>
 		<geometry>
-			<mesh filename="package://p2os_urdf/meshes/p3at_meshes/${suffix}_hubcap.stl"/>
+			<mesh filename="package://my_p2os/meshes/p3at_meshes/${suffix}_hubcap.stl"/>
 		</geometry>
 	</collision>
@@ -303,5 +303,5 @@
 		<origin xyz="0 0 0" rpy="0 0 0"/>
 		<geometry name="pioneer_geom">
-			<mesh filename="package://p2os_urdf/meshes/p3at_meshes/wheel.stl"/>
+			<mesh filename="package://my_p2os/meshes/p3at_meshes/wheel.stl"/>
 		</geometry>
 		<material name="WheelBlack"/>
@@ -310,5 +310,5 @@
 		<origin xyz="0 0 0" rpy="${-3.1415927/2} 0 0"/>
 		<geometry>
-	    <!--mesh filename="package://p2os_urdf/meshes/p3at_meshes/wheel.stl"/-->
+	    <!--mesh filename="package://my_p2os/meshes/p3at_meshes/wheel.stl"/-->
 	    <cylinder radius="0.111" length="0.075"/>
 		</geometry>
@@ -351,5 +351,5 @@
   <plugin name="controller" filename="libcontroller.so">
     <updateRate>100.0</updateRate>
-    <robotNamespace>/</robotNamespace>
+    <robotNamespace>$(arg namespace)</robotNamespace>
     <leftFrontJoint>p3at_front_left_wheel_joint</leftFrontJoint>
     <rightFrontJoint>p3at_front_right_wheel_joint</rightFrontJoint>
@@ -358,9 +358,9 @@
     <wheelSeparation>0.4</wheelSeparation>
     <wheelDiameter>0.215</wheelDiameter>
-    <robotBaseFrame>base_link</robotBaseFrame>
+    <robotBaseFrame>$(arg namespace)/base_link</robotBaseFrame>
     <torque>200</torque>
-    <topicName>cmd_vel</topicName>
-    <odometryTopic>odom</odometryTopic>
-    <odometryFrame>odom</odometryFrame>
+    <topicName>$(arg namespace)/cmd_vel</topicName>
+    <odometryTopic>$(arg namespace)/odom</odometryTopic>
+    <odometryFrame>$(arg namespace)/odom</odometryFrame>
     <broadcastTF>1</broadcastTF>
   </plugin>
